File: narcise/narcise.sch (KiCad schematic (older format))
At the start: 7 parts

Commit message: After PCB order
Parts:
- removed U?: ariadne-rescue_OKI-78SR-5v-OpenSourceCelluloid-up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, symbol ariadne-v3-cache:ariadne-rescue_OKI-78SR-5v-OpenSourceCelluloid-upuaut-rescue
- added J1, J2, J3, J6, J7, J8: 5-5530843-0, kicad-libraries:TE_5-5530843-0, symbol 5-5530843-0:5-5530843-0
- added Murata-Ceramic-Capacitor-50v1-22uF1, Murata-Ceramic-Capacitor-50v1-22uF2: C, Capacitor_THT:C_Disc_D3.0mm_W1.6mm_P2.50mm, symbol Device:C
- added Q10, Q11, Q2, Q3, Q4, Q5, Q7, Q8, Q9: IRLZ44N-horizontal, Package_TO_SOT_THT:TO-220-3_Horizontal_TabDown, symbol narcise:IRLZ44N-horizontal
- added R1, R10, R11, R2, R3, R4, R5, R7, R8, R9: R, Resistor_THT:R_Axial_DIN0204_L3.6mm_D1.6mm_P7.62mm_Horizontal, symbol Device:R
- added U1, U12, U13, U14, U2, U24, U25, U26, U3, U6, U8, U9: fpc-connector-mosfet-drain, ffc-fpc:Molex_200528-0040_1x04-1MP_P1.00mm_Horizontal, symbol narcise:fpc-connector
- added U10: OKI-78SR-5v, Converter_DCDC:Converter_DCDC_muRata_OKI-78SR_Vertical, symbol ariadne-rescue:OKI-78SR-5v-OpenSourceCelluloid-upuaut-rescue
- added U29, U30, U35, U4, U5, U7: fpc-connector-VIN, ffc-fpc:Molex_200528-0040_1x04-1MP_P1.00mm_Horizontal, symbol narcise:fpc-connector
- added X1, X10, X11, X12, X13, X14, X15, X16, X17, X18, X19, X2, X20, X21, X22, X23, X24, X25, X26, X27, X28, X29, X3, X30, X31, X32, X33, X34, X35, X36, X37, X38, X4, X5, X6, X7, X8, X9: 2059-301_998-403, P-2059-301:998-403, symbol 2059-301_998-403:2059-301_998-403
- Q1: renamed from Q?; footprint Package_TO_SOT_THT:TO-220-3_Vertical -> Package_TO_SOT_THT:TO-220-3_Horizontal_TabDown
- gave numbers to parts that had none: 5
Connections:
- net labels added: +24V, +5V, sheet1, sheet10, sheet2, sheet3, sheet4, sheet5, sheet6, sheet7, sheet8, sheet9
- net labels removed: +36V, VIN+Master1, VIN+Master2, VIN-Master1, VIN-Master2
- wire segments 17 -> 334
- no-connect marks 1 -> 7
Other:
- note added: "5V voltage regulator\n\n"
- note added: "fpc sheet\n"
- note added: "fpc-wago node\n"
- note added: "layer"
- note added: "parallell"
- note added: "perpendicular\n"
- note added: "sheet\n"
- note added: "wago node"
- note added: "wago sheet\n"
- moved on the sheet: D1, Q1, Q6, R6, U11, U21

Commit message: troubleshooting
Parts:
- J1, J2, J3, J6, J7, J8: symbol 5-5530843-0:5-5530843-0 -> narcise-rescue:5-5530843-0-5-5530843-0
- X1, X10, X11, X12, X13, X14, X15, X16, X17, X18, X19, X2, X20, X21, X22, X23, X24, X25, X26, X27, X28, X29, X3, X30, X31, X32, X33, X34, X35, X36, X37, X38, X4, X5, X6, X7, X8, X9: symbol 2059-301_998-403:2059-301_998-403 -> narcise-rescue:2059-301_998-403-2059-301_998-403
Changed lines of the file:
@@
 	10400 10900 13700 10900
 $Comp
-L 5-5530843-0:5-5530843-0 J1
+L narcise-rescue:5-5530843-0-5-5530843-0 J1
 U 1 1 604E1C17
 P 11600 10100
@@
 	12000 10600 11200 10600
 $Comp
-L 5-5530843-0:5-5530843-0 J6
+L narcise-rescue:5-5530843-0-5-5530843-0 J6
 U 1 1 6050BA30
 P 12900 10100
@@
 	10400 15500 13700 15500
 $Comp
-L 5-5530843-0:5-5530843-0 J3
+L narcise-rescue:5-5530843-0-5-5530843-0 J3
 U 1 1 605286AC
 P 11600 14700
@@
 	12000 15200 11200 15200
 $Comp
-L 5-5530843-0:5-5530843-0 J8
+L narcise-rescue:5-5530843-0-5-5530843-0 J8
 U 1 1 605286BE
 P 12900 14700
@@
 	10400 13150 13700 13150
 $Comp
-L 5-5530843-0:5-5530843-0 J2
+L narcise-rescue:5-5530843-0-5-5530843-0 J2
 U 1 1 6053912E
 P 11600 12350
@@
 	12000 12850 11200 12850
 $Comp
-L 5-5530843-0:5-5530843-0 J7
+L narcise-rescue:5-5530843-0-5-5530843-0 J7
 U 1 1 60539140
 P 12900 12350
@@
 	10400 11100 10400 13150
 $Comp
-L 2059-301_998-403:2059-301_998-403 X6
+L narcise-rescue:2059-301_998-403-2059-301_998-403 X6
 U 1 1 6047B3DE
 P 2900 5800
@@
 Connection ~ 2700 5800
 $Comp
-L 2059-301_998-403:2059-301_998-403 X3
+L narcise-rescue:2059-301_998-403-2059-301_998-403 X3
 U 1 1 604A484B
 P 2600 7950
@@
 Connection ~ 2400 7950
 $Comp
-L 2059-301_998-403:2059-301_998-403 X23
+L narcise-rescue:2059-301_998-403-2059-301_998-403 X23
 U 1 1 6050C39F
 P 13850 7400
@@
 $EndComp
 $Comp
-L 2059-301_998-403:2059-301_998-403 X24
+L narcise-rescue:2059-301_998-403-2059-301_998-403 X24
 U 1 1 6050CB28
 P 13850 7800
@@
 $EndComp
 $Comp
-L 2059-301_998-403:2059-301_998-403 X30
+L narcise-rescue:2059-301_998-403-2059-301_998-403 X30
 U 1 1 6054402C
 P 18550 9000
@@
 fpc-wago node\n
 $Comp
-L 2059-301_998-403:2059-301_998-403 X27
+L narcise-rescue:2059-301_998-403-2059-301_998-403 X27
 U 1 1 605A5804
 P 17250 1200
@@
 wago sheet\n
 $Comp
-L 2059-301_998-403:2059-301_998-403 X33
+L narcise-rescue:2059-301_998-403-2059-301_998-403 X33
 U 1 1 605A5E2F
 P 18950 1200
@@
 sheet10
 $Comp
-L 2059-301_998-403:2059-301_998-403 X28
+L narcise-rescue:2059-301_998-403-2059-301_998-403 X28
 U 1 1 6066CD66
 P 17250 2350
@@
 wago sheet\n
 $Comp
-L 2059-301_998-403:2059-301_998-403 X34
+L narcise-rescue:2059-301_998-403-2059-301_998-403 X34
 U 1 1 6066CD70
 P 18950 2350
@@
 	20300 2850 16550 2850
 $Comp
-L 2059-301_998-403:2059-301_998-403 X29
+L narcise-rescue:2059-301_998-403-2059-301_998-403 X29
 U 1 1 6067FD4C
 P 17250 3500
@@
 wago sheet\n
 $Comp
-L 2059-301_998-403:2059-301_998-403 X35
+L narcise-rescue:2059-301_998-403-2059-301_998-403 X35
 U 1 1 6067FD56
 P 18950 3500
@@
 $EndComp
 $Comp
-L 2059-301_998-403:2059-301_998-403 X31
+L narcise-rescue:2059-301_998-403-2059-301_998-403 X31
 U 1 1 60740120
 P 18550 10950
@@
 $EndComp
 $Comp
-L 2059-301_998-403:2059-301_998-403 X32
+L narcise-rescue:2059-301_998-403-2059-301_998-403 X32
 U 1 1 608C3019
 P 18550 12850
@@
 fpc-wago node\n
 $Comp
-L 2059-301_998-403:2059-301_998-403 X21
+L narcise-rescue:2059-301_998-403-2059-301_998-403 X21
 U 1 1 608DF830
 P 13850 5750
@@
 $EndComp
 $Comp
-L 2059-301_998-403:2059-301_998-403 X22
+L narcise-rescue:2059-301_998-403-2059-301_998-403 X22
 U 1 1 608DF836
 P 13850 6150
@@
 wago node
 $Comp
-L 2059-301_998-403:2059-301_998-403 X25
+L narcise-rescue:2059-301_998-403-2059-301_998-403 X25
 U 1 1 608F4B56
 P 14700 9100
@@
 $EndComp
 $Comp
-L 2059-301_998-403:2059-301_998-403 X26
+L narcise-rescue:2059-301_998-403-2059-301_998-403 X26
 U 1 1 608F4B5C
 P 14700 9500
@@
 layer
 $Comp
-L 2059-301_998-403:2059-301_998-403 X10
+L narcise-rescue:2059-301_998-403-2059-301_998-403 X10
 U 1 1 60A66737
 P 5800 5800
@@
 Connection ~ 5600 5800
 $Comp
-L 2059-301_998-403:2059-301_998-403 X7
+L narcise-rescue:2059-301_998-403-2059-301_998-403 X7
 U 1 1 60A66740
 P 5500 7950
@@
 layer
 $Comp
-L 2059-301_998-403:2059-301_998-403 X4
+L narcise-rescue:2059-301_998-403-2059-301_998-403 X4
 U 1 1 60A75046
 P 2850 8800
@@
 Connection ~ 2650 8800
 $Comp
-L 2059-301_998-403:2059-301_998-403 X1
+L narcise-rescue:2059-301_998-403-2059-301_998-403 X1
 U 1 1 60A7504F
 P 2550 10950
@@
 layer
 $Comp
-L 2059-301_998-403:2059-301_998-403 X11
+L narcise-rescue:2059-301_998-403-2059-301_998-403 X11
 U 1 1 60A852F7
 P 5800 8800
@@
 Connection ~ 5600 8800
 $Comp
-L 2059-301_998-403:2059-301_998-403 X8
+L narcise-rescue:2059-301_998-403-2059-301_998-403 X8
 U 1 1 60A85300
 P 5500 10950
@@
 layer
 $Comp
-L 2059-301_998-403:2059-301_998-403 X5
+L narcise-rescue:2059-301_998-403-2059-301_998-403 X5
 U 1 1 60AB7D15
 P 2850 11850
@@
 Connection ~ 2650 11850
 $Comp
-L 2059-301_998-403:2059-301_998-403 X2
+L narcise-rescue:2059-301_998-403-2059-301_998-403 X2
 U 1 1 60AB7D1E
 P 2550 14000
@@
 layer
 $Comp
-L 2059-301_998-403:2059-301_998-403 X12
+L narcise-rescue:2059-301_998-403-2059-301_998-403 X12
 U 1 1 60ACC1F3
 P 5800 11900
@@
 Connection ~ 5600 11900
 $Comp
-L 2059-301_998-403:2059-301_998-403 X9
+L narcise-rescue:2059-301_998-403-2059-301_998-403 X9
 U 1 1 60ACC1FC
 P 5500 14050
@@
 layer
 $Comp
-L 2059-301_998-403:2059-301_998-403 X16
+L narcise-rescue:2059-301_998-403-2059-301_998-403 X16
 U 1 1 60B03EC3
 P 8700 5800
@@
 Connection ~ 8500 5800
 $Comp
-L 2059-301_998-403:2059-301_998-403 X13
+L narcise-rescue:2059-301_998-403-2059-301_998-403 X13
 U 1 1 60B03ECC
 P 8400 7950
@@
 layer
 $Comp
-L 2059-301_998-403:2059-301_998-403 X17
+L narcise-rescue:2059-301_998-403-2059-301_998-403 X17
 U 1 1 60B1B95A
 P 8750 8800
@@
 Connection ~ 8550 8800
 $Comp
-L 2059-301_998-403:2059-301_998-403 X14
+L narcise-rescue:2059-301_998-403-2059-301_998-403 X14
 U 1 1 60B1B963
 P 8450 10950
@@
 layer
 $Comp
-L 2059-301_998-403:2059-301_998-403 X18
+L narcise-rescue:2059-301_998-403-2059-301_998-403 X18
 U 1 1 60B34FB5
 P 8750 11900
@@
 Connection ~ 8550 11900
 $Comp
-L 2059-301_998-403:2059-301_998-403 X15
+L narcise-rescue:2059-301_998-403-2059-301_998-403 X15
 U 1 1 60B34FBE
 P 8450 14050
@@
 layer
 $Comp
-L 2059-301_998-403:2059-301_998-403 X20
+L narcise-rescue:2059-301_998-403-2059-301_998-403 X20
 U 1 1 60B500A7
 P 11600 5800
@@
 Connection ~ 11400 5800
 $Comp
-L 2059-301_998-403:2059-301_998-403 X19
+L narcise-rescue:2059-301_998-403-2059-301_998-403 X19
 U 1 1 60B500B0
 P 11300 7950
@@
 $EndComp
 $Comp
-L 2059-301_998-403:2059-301_998-403 X36
+L narcise-rescue:2059-301_998-403-2059-301_998-403 X36
 U 1 1 60BEEE20
 P 21150 9000
@@
 $EndComp
 $Comp
-L 2059-301_998-403:2059-301_998-403 X37
+L narcise-rescue:2059-301_998-403-2059-301_998-403 X37
 U 1 1 60BEEE34
 P 21150 10950
@@
 $EndComp
 $Comp
-L 2059-301_998-403:2059-301_998-403 X38
+L narcise-rescue:2059-301_998-403-2059-301_998-403 X38
 U 1 1 60BEEE48
 P 21150 12850
